File: instrumentation_amplifier/instrument_amplifier/instrument_amplifier.kicad_sch (KiCad schematic)
At the start: 20 parts, among them J1 Conn_01x06_Pin, U1 LM324, U2 LM324

Commit message: final commit, ready to fab
Parts:
- added H1, H2, H3, H4: MountingHole_Pad, MountingHole:MountingHole_2.5mm_Pad, symbol Mechanical:MountingHole_Pad
- J1: footprint Connector_PinHeader_1.00mm:PinHeader_1x07_P1.00mm_Horizontal -> Connector_PinHeader_2.54mm:PinHeader_1x06_P2.54mm_Horizontal
Connections:
- net E+: now also J1.4 (Pin_4); no longer J1.3 (Pin_3)
- net E-: now also J1.3 (Pin_3); no longer J1.4 (Pin_4)
- net GND: now also H1.1, H2.1, H3.1, H4.1
